Commit message: Run model in gazebo

File: my_rb1_description/urdf/my_rb1_robot.urdf (robot description, URDF)
Before this commit: robot rb1_robot, 7 links, 6 joints
Links:
- link back_caster: mass 0.5 -> 1.5; geometry collision cylinder length=.010 radius=.025; visual cylinder length=0.10 radius=.025
- link base_link: mass 19 -> 16
- link front_caster: mass 0.5 -> 1.5; geometry collision cylinder length=.010 radius=.025; visual cylinder length=.010 radius=.025
- link front_laser: mass 1 -> 2
- link left_wheel: geometry collision cylinder length=.020 radius=.025; visual cylinder length=.020 radius=.025

Commit message: add driver control and laserplugins

File: my_rb1_description/urdf/my_rb1_robot.urdf (robot description, URDF)
Before this commit: robot rb1_robot, 7 links, 6 joints
Links:
- link back_caster: geometry collision sphere radius=0.025; visual sphere radius=0.025
- link front_caster: geometry collision sphere radius=0.025; visual sphere radius=0.025
- link right_wheel: geometry collision cylinder length=.020 radius=.025; visual cylinder length=.020 radius=.025
Joints:
- joint base_link_back_caster_joint: axis 0 1 0 -> 0 1 1; origin xyz=0.1 0 -0.15 rpy=1.57 0 0  -> xyz=0.1 0 -0.15 rpy=0 0 0 ; type fixed -> continuous
- joint base_link_front_caster_joint: axis 0 0 0 -> 0 1 1; type fixed -> continuous

Commit message: modify robot caster wheel

File: my_rb1_description/urdf/my_rb1_robot.urdf (robot description, URDF)
Before this commit: robot rb1_robot, 7 links, 6 joints
Links:
- link back_caster: mass 1.5 -> 1; geometry collision sphere radius=.025; visual sphere radius=.025
- link front_caster: mass 1.5 -> 1; geometry collision sphere radius=.025; visual sphere radius=.025
- link front_laser: mass 2 -> 1
- link left_wheel: mass 2 -> 3
- link right_wheel: mass 2 -> 3
Joints:
- joint base_link_back_caster_joint: axis 0 1 1 -> 0 1 0; origin xyz=0.1 0 -0.15 rpy=0 0 0  -> xyz=-0.1 0 -0.15 rpy=1.57 0 0 ; type continuous -> fixed
- joint base_link_front_caster_joint: axis 0 1 1 -> 0 0 0; origin xyz=-0.1 0 -0.15 rpy=1.57 0 0  -> xyz=0.1 0 -0.15 rpy=1.57 0 0 ; type continuous -> fixed
- joint base_link_plate_joint: origin xyz=0 0 0 rpy=0 0 0 -> xyz=0 0 -0.15 rpy=0 0 0

Commit message: change wheel rotation direction

File: my_rb1_description/urdf/my_rb1_robot.urdf (robot description, URDF)
Before this commit: robot rb1_robot, 7 links, 6 joints
Joints:
- joint base_link_left_wheel_joint: axis 0 0 1 -> 0 0 -1; origin xyz=0 -0.2 -0.15 rpy=1.57 0 0  -> xyz=0 0.2 -0.15 rpy=1.57 0 0 
- joint base_link_right_wheel_joint: axis 0 0 1 -> 0 0 -1; origin xyz=0 0.2 -0.15 rpy=1.57 0 0  -> xyz=0 -0.2 -0.15 rpy=1.57 0 0 
